Commit message: Add new mesh assets for parts 228-2500-2000, 228-2500-208, and 228-2500-209
- Added JSON configuration files for parts 228-2500-2000, 228-2500-208, and 228-2500-209.
- Included corresponding STL files for each part, with sizes of 1053 KB, 4766 KB, and 2114 KB respectively.
- All parts are marked as non-standard content and are associated with part ID "JFD".

File: src/py_package/meshes/robot.urdf (robot description, URDF)
Before this commit: robot meshes, 5 links, 4 joints
Links:
- removed link fl
- removed link fr
- removed link rl
- removed link rr
- added link 228_2500_208, mass 1e-09; collision mesh filename=file:///home/menglin/ROS2/src/py_package/meshes/assets/228_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; collision mesh filename=file:///home/menglin/ROS2/src/py_package/meshes/assets/228_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
- added link 228_2500_208_2, mass 1e-09; collision mesh filename=file:///home/menglin/ROS2/src/py_package/meshes/assets/228_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; collision mesh filename=file:///home/menglin/ROS2/src/py_package/meshes/assets/228_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
- added link 228_2500_208_3, mass 1e-09; collision mesh filename=file:///home/menglin/ROS2/src/py_package/meshes/assets/228_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; collision mesh filename=file:///home/menglin/ROS2/src/py_package/meshes/assets/228_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
- added link 228_2500_209, mass 1e-09; collision mesh filename=file:///home/menglin/ROS2/src/py_package/meshes/assets/228_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; collision mesh filename=file:///home/menglin/ROS2/src/py_package/meshes/assets/228_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
- added link 228_2500_209_2, mass 1e-09; collision mesh filename=file:///home/menglin/ROS2/src/py_package/meshes/assets/228_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; collision mesh filename=file:///home/menglin/ROS2/src/py_package/meshes/assets/228_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
- added link 228_2500_209_3, mass 1e-09; collision mesh filename=file:///home/menglin/ROS2/src/py_package/meshes/assets/228_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; collision mesh filename=file:///home/menglin/ROS2/src/py_package/meshes/assets/228_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
- link base_link: mass 2.65759 -> 1e-09; geometry collision mesh filename=file:///home/menglin/ROS2/src/py_package/meshes/assets/228_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; collision mesh filename=file:///home/menglin/ROS2/src/py_package/meshes/assets/228_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
Joints:
- removed joint fl
- removed joint fr
- removed joint rl
- removed joint rr
- added joint w0: type revolute, parent base_link, child 228_2500_208_3, origin xyz=-0.00276906 -0.0749443 -0.033147 rpy=-1.5708 -5.1944e-08 -5.4078e-08, axis 0 0 1, limit lower=-3.141592653589793 upper=3.141592653589793 effort=10 velocity=10
- added joint w1: type revolute, parent base_link, child 228_2500_209_3, origin xyz=0.0548464 -0.04168 -0.033147 rpy=-2.61799 1.5708 0, axis 0 0 1, limit lower=-3.141592653589793 upper=3.141592653589793 effort=10 velocity=10
- added joint w2: type revolute, parent base_link, child 228_2500_208_2, origin xyz=0.0539804 0.0243486 -0.033147 rpy=0.523599 -1.5708 0, axis 0 0 1, limit lower=-3.141592653589793 upper=3.141592653589793 effort=10 velocity=10
- added joint w3: type revolute, parent base_link, child 228_2500_209_2, origin xyz=-0.00276905 0.0581129 -0.033147 rpy=1.5708 -5.1944e-08 -5.4078e-08, axis 0 0 1, limit lower=-3.141592653589793 upper=3.141592653589793 effort=10 velocity=10
- added joint w4: type revolute, parent base_link, child 228_2500_209, origin xyz=-0.0603845 0.0248486 -0.033147 rpy=2.61799 -1.5708 0, axis 0 0 1, limit lower=-3.141592653589793 upper=3.141592653589793 effort=10 velocity=10
- added joint w5: type revolute, parent base_link, child 228_2500_208, origin xyz=-0.0603845 -0.04168 -0.033147 rpy=-1.5708 -6.0447e-08 -1.0472, axis 0 0 1, limit lower=-3.141592653589793 upper=3.141592653589793 effort=10 velocity=10

Commit message: import robot arm model

File: src/py_package/meshes/robot.urdf (robot description, URDF)
Before this commit: robot meshes, 7 links, 6 joints
Links:
- removed link 228_2500_208
- removed link 228_2500_208_2
- removed link 228_2500_208_3
- removed link 228_2500_209
- removed link 228_2500_209_2
- removed link 228_2500_209_3
- added link arm1, mass 6.76494; collision mesh filename=file:///home/menglin/ROS2/src/py_package/meshes/assets/arm1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; visual mesh filename=file:///home/menglin/ROS2/src/py_package/meshes/assets/arm1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
- added link arm1_base, mass 7.44232; collision mesh filename=file:///home/menglin/ROS2/src/py_package/meshes/assets/arm1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; visual mesh filename=file:///home/menglin/ROS2/src/py_package/meshes/assets/arm1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
- added link arm2, mass 6.76494; collision mesh filename=file:///home/menglin/ROS2/src/py_package/meshes/assets/arm2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; visual mesh filename=file:///home/menglin/ROS2/src/py_package/meshes/assets/arm2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
- added link arm2_base, mass 6.08574; collision mesh filename=file:///home/menglin/ROS2/src/py_package/meshes/assets/arm2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; visual mesh filename=file:///home/menglin/ROS2/src/py_package/meshes/assets/arm2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
- link base_link: mass 1e-09 -> 116.707; geometry collision mesh filename=file:///home/menglin/ROS2/src/py_package/meshes/assets/base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; visual mesh filename=file:///home/menglin/ROS2/src/py_package/meshes/assets/base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
Joints:
- removed joint w0
- removed joint w1
- removed joint w2
- removed joint w3
- removed joint w4
- removed joint w5
- added joint arm1: type revolute, parent arm1_base, child arm1, origin xyz=0.0536635 0 -0.87 rpy=-0 1.5708 0, axis 0 0 1, limit lower=-3.141592653589793 upper=3.141592653589793 effort=10 velocity=10
- added joint arm1_base: type revolute, parent base_link, child arm1_base, origin xyz=-0 0 0.1 rpy=-3.14159 -0 0, axis 0 0 1, limit lower=-3.141592653589793 upper=3.141592653589793 effort=10 velocity=10
- added joint arm2: type revolute, parent arm2_base, child arm2, origin xyz=0.0536635 -0 -0.87 rpy=-3.14159 1.5708 0, axis 0 0 1, limit lower=-3.141592653589793 upper=3.141592653589793 effort=10 velocity=10
- added joint arm2_base: type revolute, parent arm1, child arm2_base, origin xyz=0.085 -0 -0.0536656 rpy=3.14159 1.5708 0, axis 0 0 1, limit lower=-3.141592653589793 upper=3.141592653589793 effort=10 velocity=10
