Commit message: Add arm3_base part configuration and STL file
- Created a new JSON configuration file for the arm3_base part, including essential metadata such as document ID, element ID, and part ID.
- Added the corresponding STL file for the arm3_base part, which is essential for 3D modeling and rendering.

File: src/py_package/meshes/robot.urdf (robot description, URDF)
Before this commit: robot meshes, 5 links, 4 joints
Links:
- added link arm3, mass 3.63498; collision mesh filename=file:///home/menglin/ROS2/src/py_package/meshes/assets/arm3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; visual mesh filename=file:///home/menglin/ROS2/src/py_package/meshes/assets/arm3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
- added link arm3_base, mass 5.49197; collision mesh filename=file:///home/menglin/ROS2/src/py_package/meshes/assets/arm3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; visual mesh filename=file:///home/menglin/ROS2/src/py_package/meshes/assets/arm3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
- link arm1: mass 6.76494 -> 6.6886
- link arm1_base: mass 7.44232 -> 3.45791
- link arm2: mass 6.76494 -> 6.6886
- link arm2_base: mass 6.08574 -> 5.49197
- link base_link: mass 116.707 -> 130.02
Joints:
- added joint arm3: type revolute, parent arm3_base, child arm3, origin xyz=-0.0536635 0 -0.08 rpy=3.14159 1.5708 0, axis 0 0 1, limit lower=-3.141592653589793 upper=3.141592653589793 effort=10 velocity=10
- added joint arm3_base: type revolute, parent arm2, child arm3_base, origin xyz=0.825 -0 -0.0536656 rpy=-3.14159 1.5708 0, axis 0 0 1, limit lower=-3.141592653589793 upper=3.141592653589793 effort=10 velocity=10
- joint arm1: origin xyz=0.0536635 0 -0.87 rpy=-0 1.5708 0 -> xyz=-0.0536635 0 -0.18 rpy=3.14159 1.5708 0
- joint arm1_base: origin xyz=-0 0 0.1 rpy=-3.14159 -0 0 -> xyz=0 0 0.14 rpy=3.14159 0 0
- joint arm2: origin xyz=0.0536635 -0 -0.87 rpy=-3.14159 1.5708 0 -> xyz=-0.0536635 0 -0.08 rpy=-3.14159 1.5708 0
- joint arm2_base: origin xyz=0.085 -0 -0.0536656 rpy=3.14159 1.5708 0 -> xyz=0.825 -0 -0.0536656 rpy=3.14159 1.5708 0
